File: phase_chan.kicad_sch (KiCad schematic)
At the start: 0 parts

Commit message: sch_0v1 ready for review
Parts:
- added C25, C26, C27, C28: C, symbol Device:C
- added J2, J4: Conn_Coaxial, symbol Connector:Conn_Coaxial
- added L3, L4: L, symbol Device:L
- added U6: ~, symbol generated_symbols:JSPHS-x+
Connections:
- new net: C26.1, L3.2, U6.1 (IN)
- new net: C28.1, L4.2, U6.7 (OUT)
- new net: C25.1, J2.1 (In), L3.1
- new net: C27.1, J4.1 (In), L4.1
- new net GND: C25.2, C26.2, C27.2, C28.2, J2.2 (Ext), J4.2 (Ext), U6.10 (GND), U6.11 (GND), U6.12 (GND), U6.13 (GND), U6.14 (GND), U6.2 (GND), U6.3 (GND), U6.5 (GND), U6.8 (GND), U6.9 (GND)
- new net VBIAS: U6.4 (CTL), U6.6 (CTL)
